Commit message: Add torso to pinchy

File: pinchy_robot/urdf/pinchy.urdf (robot description, URDF)
Before this commit: robot pinchy, 2 links, 1 joints
Links:
- added link torso; visual cylinder length=0.5 radius=0.05
Joints:
- added joint base_link_to_torso: type continuous, parent base_link, child torso, origin xyz=0 0 0.05 rpy=0 0 0, axis 0 0 1

Commit message: Add arms to pinchy

File: pinchy_robot/urdf/pinchy.urdf (robot description, URDF)
Before this commit: robot pinchy, 3 links, 2 joints
Links:
- added link lower_arm; visual cylinder length=0.4 radius=0.05
- added link upper_arm; visual cylinder length=0.4 radius=0.05
Joints:
- added joint torso_to_upper_arm: type continuous, parent torso, child upper_arm, origin xyz=0 -0.1 0.45 rpy=0 1.5708 0, axis 0 1 0
- added joint upper_arm_to_lower_arm: type continuous, parent upper_arm, child lower_arm, origin xyz=0 0.1 0.35 rpy=0 0 0, axis 0 1 0

Commit message: Add hand to pinchy

File: pinchy_robot/urdf/pinchy.urdf (robot description, URDF)
Before this commit: robot pinchy, 5 links, 4 joints
Links:
- added link hand; visual box size=0.05 0.05 0.05
Joints:
- added joint lower_arm_to_hand: type continuous, parent lower_arm, child hand, origin xyz=0 0 0.425 rpy=0 0 0, axis 0 1 0

Commit message: add collision and inertia to urdf

File: pinchy_robot/urdf/pinchy.urdf (robot description, URDF)
Before this commit: robot pinchy, 6 links, 5 joints
Links:
- link base_link: mass None -> 1.0; geometry collision cylinder length=0.05 radius=0.1; visual cylinder length=0.05 radius=0.1
- link hand: mass None -> 1.0; geometry collision box size=0.05 0.05 0.05; visual box size=0.05 0.05 0.05
- link lower_arm: mass None -> 1.0; geometry collision cylinder length=0.4 radius=0.05; visual cylinder length=0.4 radius=0.05
- link torso: mass None -> 1.0; geometry collision cylinder length=0.5 radius=0.05; visual cylinder length=0.5 radius=0.05
- link upper_arm: mass None -> 1.0; geometry collision cylinder length=0.4 radius=0.05; visual cylinder length=0.4 radius=0.05
