Commit message: Use the urdf file instead of sdf for now

File: pinchy_robot/pinchy_robot_description/models/pinchy/pinchy.urdf (robot description, URDF)
Before this commit: robot pinchy, 6 links, 5 joints
Links:
- removed link world
- added link massive_block, mass 1000.0; collision box size=1 1 0.0001; visual box size=1 1 0.0001
- added link root
Joints:
- removed joint world_to_base_link
- added joint massive_block_to_base_link: type fixed, parent massive_block, child base_link
- added joint root_to_massive_block: type fixed, parent root, child massive_block

Commit message: make block smaller

File: pinchy_robot/pinchy_robot_description/models/pinchy/pinchy.urdf (robot description, URDF)
Before this commit: robot pinchy, 7 links, 6 joints
Links:
- link massive_block: geometry collision box size=0.1 0.1 0.0001; visual box size=0.1 0.1 0.0001
