Commit message: playing around with xacro and urdf files

File: pinchy_robot/pinchy_robot_description/models/pinchy/pinchy_core.xacro (robot description, xacro)
@@ -1,23 +1,16 @@
-<?xml version="1.0" ?>
-<!-- =================================================================================== -->
-<!-- |    This document was autogenerated by xacro from pinchy.urdf.xacro              | -->
-<!-- |    EDITING THIS FILE BY HAND IS NOT RECOMMENDED                                 | -->
-<!-- =================================================================================== -->
-<robot name="pinchy">
+<?xml version="1.0"?>
+<robot xmlns:xacro="http://www.ros.org/wiki/xacro">
   <material name="silver">
     <color rgba="0.75 0.75 0.75 1"/>
   </material>
-  <material name="invisible">
-    <color rgba="0 0 0 0"/>
-  </material>
-  <link name="root"/>
-  <link name="massive_block">
-    <visual name="massive_block_visual">
+  <link name='root'/>
+  <link name='massive_block'>
+    <visual>
       <geometry>
         <box size="0.1 0.1 0.0001"/>
       </geometry>
-      <material name="invisible"/>
+      <material name="silver"/>
     </visual>
-    <collision name="massive_block_collision">
+    <collision>
       <pose>0 0 0 0 0 0</pose>
       <geometry>
@@ -28,5 +21,6 @@
       <mass value="1000.0"/>
       <origin xyz="0 0 0"/>
-      <inertia ixx="0" ixy="0" ixz="0" iyy="0" iyz="0" izz="0"/>
+      <inertia ixx="0" iyy="0" izz="0"
+        ixy="0" ixz="0" iyz="0"/>
     </inertial>
   </link>
@@ -52,5 +46,6 @@
       <mass value="1.0"/>
       <origin xyz="0 0 0.025"/>
-      <inertia ixx="0.0027" ixy="0" ixz="0" iyy="0.0027" iyz="0" izz="0.005"/>
+      <inertia ixx="0.0027" iyy="0.0027" izz="0.005"
+        ixy="0" ixz="0" iyz="0"/>
     </inertial>
   </link>
@@ -76,5 +71,6 @@
       <mass value="1.0"/>
       <origin xyz="0 0 0.25"/>
-      <inertia ixx="0.002146" ixy="0" ixz="0" iyy="0.002146" iyz="0" izz="0.00125"/>
+      <inertia ixx="0.002146" iyy="0.002146" izz="0.00125"
+        ixy="0" ixz="0" iyz="0"/>
     </inertial>
   </link>
@@ -102,5 +98,6 @@
       <mass value="1.0"/>
       <origin xyz="0 0 0.2"/>
-      <inertia ixx="0.01396" ixy="0" ixz="0" iyy="0.01396" iyz="0" izz="0.00125"/>
+      <inertia ixx="0.01396" iyy="0.01396" izz="0.00125"
+        ixy="0" ixz="0" iyz="0"/>
     </inertial>
   </link>
@@ -128,5 +125,6 @@
       <mass value="1.0"/>
       <origin xyz="0 0 0.2"/>
-      <inertia ixx="0.01396" ixy="0" ixz="0" iyy="0.01396" iyz="0" izz="0.00125"/>
+      <inertia ixx="0.01396" iyy="0.01396" izz="0.00125"
+        ixy="0" ixz="0" iyz="0"/>
     </inertial>
   </link>
@@ -151,5 +149,6 @@
     <inertial>
       <mass value="1.0"/>
-      <inertia ixx="0.00042" ixy="0" ixz="0" iyy="0.00042" iyz="0" izz="0.00042"/>
+      <inertia ixx="0.00042" iyy="0.00042" izz="0.00042"
+        ixy="0" ixz="0" iyz="0"/>
     </inertial>
   </link>
