Commit message: refactor models and launch files to get ready for ros2_control

File: pinchy_robot/pinchy_robot_description/models/pinchy_description.urdf.xacro (robot description, xacro)
@@ -1,31 +1,9 @@
 <?xml version="1.0"?>
 <robot xmlns:xacro="http://www.ros.org/wiki/xacro">
-  <material name="silver">
-    <color rgba="0.75 0.75 0.75 1"/>
-  </material>
-  <link name='root'/>
-  <link name='massive_block'>
-    <visual>
-      <geometry>
-        <box size="0.1 0.1 0.0001"/>
-      </geometry>
-      <material name="silver"/>
-    </visual>
-    <collision>
-      <pose>0 0 0 0 0 0</pose>
-      <geometry>
-        <box size="0.1 0.1 0.0001"/>
-      </geometry>
-    </collision>
-    <inertial>
-      <mass value="1000.0"/>
-      <origin xyz="0 0 0"/>
-      <inertia ixx="0" iyy="0" izz="0"
-        ixy="0" ixz="0" iyz="0"/>
-    </inertial>
-  </link>
-  <joint name="root_to_massive_block" type="fixed">
-    <parent link="root"/>
-    <child link="massive_block"/>
+  <xacro:macro name="pinchy" params="parent *origin">
+  <joint name="base_joint" type="fixed">
+    <xacro:insert_block name="origin" />
+    <parent link="${parent}"/>
+    <child link="base_link"/>
   </joint>
   <link name="base_link">
@@ -50,7 +28,9 @@
     </inertial>
   </link>
-  <joint name="massive_block_to_base_link" type="fixed">
-    <parent link="massive_block"/>
-    <child link="base_link"/>
+  <joint name="base_link_to_torso" type="continuous">
+    <axis xyz="0 0 1"/>
+    <parent link="base_link"/>
+    <child link="torso"/>
+    <origin rpy="0 0 0" xyz="0 0 0.05"/>
   </joint>
   <link name="torso">
@@ -75,31 +55,4 @@
     </inertial>
   </link>
-  <joint name="base_link_to_torso" type="continuous">
-    <axis xyz="0 0 1"/>
-    <parent link="base_link"/>
-    <child link="torso"/>
-    <origin rpy="0 0 0" xyz="0 0 0.05"/>
-  </joint>
-  <link name="upper_arm">
-    <visual>
-      <geometry>
-        <cylinder length="0.4" radius="0.05"/>
-      </geometry>
-      <material name="silver"/>
-      <origin xyz="0 0 0.2"/>
-    </visual>
-    <collision>
-      <geometry>
-        <cylinder length="0.4" radius="0.05"/>
-      </geometry>
-      <origin xyz="0 0 0.2"/>
-    </collision>
-    <inertial>
-      <mass value="1.0"/>
-      <origin xyz="0 0 0.2"/>
-      <inertia ixx="0.01396" iyy="0.01396" izz="0.00125"
-        ixy="0" ixz="0" iyz="0"/>
-    </inertial>
-  </link>
   <joint name="torso_to_upper_arm" type="continuous">
     <axis xyz="0 1 0"/>
@@ -108,5 +61,5 @@
     <origin rpy="0 1.5708 0" xyz="0 -0.1 0.45"/>
   </joint>
-  <link name="lower_arm">
+  <link name="upper_arm">
     <visual>
       <geometry>
@@ -135,4 +88,31 @@
     <origin rpy="0 0 0" xyz="0 0.1 0.35"/>
   </joint>
+  <link name="lower_arm">
+    <visual>
+      <geometry>
+        <cylinder length="0.4" radius="0.05"/>
+      </geometry>
+      <material name="silver"/>
+      <origin xyz="0 0 0.2"/>
+    </visual>
+    <collision>
+      <geometry>
+        <cylinder length="0.4" radius="0.05"/>
+      </geometry>
+      <origin xyz="0 0 0.2"/>
+    </collision>
+    <inertial>
+      <mass value="1.0"/>
+      <origin xyz="0 0 0.2"/>
+      <inertia ixx="0.01396" iyy="0.01396" izz="0.00125"
+        ixy="0" ixz="0" iyz="0"/>
+    </inertial>
+  </link>
+  <joint name="lower_arm_to_hand" type="continuous">
+    <axis xyz="0 1 0"/>
+    <parent link="lower_arm"/>
+    <child link="hand"/>
+    <origin rpy="0 0 0" xyz="0 0 0.425"/>
+  </joint>
   <link name="hand">
     <visual>
@@ -153,9 +133,4 @@
     </inertial>
   </link>
-  <joint name="lower_arm_to_hand" type="continuous">
-    <axis xyz="0 1 0"/>
-    <parent link="lower_arm"/>
-    <child link="hand"/>
-    <origin rpy="0 0 0" xyz="0 0 0.425"/>
-  </joint>
+  </xacro:macro>
 </robot>
