Commit message: Add onshape exported urdf

File: pinchy_robot/pinchy_robot_description/models/pinchy.urdf.xacro (robot description, xacro)
@@ -3,5 +3,6 @@
   <xacro:arg name="use_gazebo" default="false" />
   <!-- Import pinchy macro -->
-  <xacro:include filename="$(find pinchy_robot_description)/models/pinchy_description.urdf.xacro" />
+  <!-- <xacro:include filename="$(find pinchy_robot_description)/models/pinchy_description.urdf.xacro" /> -->
+  <xacro:include filename="$(find pinchy_robot_description)/models/pinchy_onshape.urdf.xacro" />
   <!-- Import pinchy Rviz colors -->
   <xacro:include filename="$(find pinchy_robot_description)/models/pinchy.materials.xacro" />

File: pinchy_robot/pinchy_robot_description/models/pinchy_description.urdf.xacro (robot description, xacro)
@@ -2,135 +2,130 @@
 <robot xmlns:xacro="http://www.ros.org/wiki/xacro">
   <xacro:macro name="pinchy" params="parent *origin">
-  <joint name="base_joint" type="fixed">
-    <xacro:insert_block name="origin" />
-    <parent link="${parent}"/>
-    <child link="base_link"/>
-  </joint>
-  <link name="base_link">
-    <visual>
-      <geometry>
-        <cylinder length="0.05" radius="0.1"/>
-      </geometry>
-      <material name="silver"/>
-      <origin xyz="0 0 0.025"/>
-    </visual>
-    <collision>
-      <geometry>
-        <cylinder length="0.05" radius="0.1"/>
-      </geometry>
-      <origin xyz="0 0 0.025"/>
-    </collision>
-    <inertial>
-      <mass value="1.0"/>
-      <origin xyz="0 0 0.025"/>
-      <inertia ixx="0.0027" iyy="0.0027" izz="0.005"
-        ixy="0" ixz="0" iyz="0"/>
-    </inertial>
-  </link>
-  <joint name="base_link_to_torso" type="continuous">
-    <axis xyz="0 0 1"/>
-    <parent link="base_link"/>
-    <child link="torso"/>
-    <origin rpy="0 0 0" xyz="0 0 0.05"/>
-  </joint>
-  <link name="torso">
-    <visual>
-      <geometry>
-        <cylinder length="0.5" radius="0.05"/>
-      </geometry>
-      <material name="silver"/>
-      <origin xyz="0 0 0.25"/>
-    </visual>
-    <collision>
-      <geometry>
-        <cylinder length="0.5" radius="0.05"/>
-      </geometry>
-      <origin xyz="0 0 0.25"/>
-    </collision>
-    <inertial>
-      <mass value="1.0"/>
-      <origin xyz="0 0 0.25"/>
-      <inertia ixx="0.002146" iyy="0.002146" izz="0.00125"
-        ixy="0" ixz="0" iyz="0"/>
-    </inertial>
-  </link>
-  <joint name="torso_to_upper_arm" type="continuous">
-    <axis xyz="0 1 0"/>
-    <parent link="torso"/>
-    <child link="upper_arm"/>
-    <origin rpy="0 1.5708 0" xyz="0 -0.1 0.45"/>
-  </joint>
-  <link name="upper_arm">
-    <visual>
-      <geometry>
-        <cylinder length="0.4" radius="0.05"/>
-      </geometry>
-      <material name="silver"/>
-      <origin xyz="0 0 0.2"/>
-    </visual>
-    <collision>
-      <geometry>
-        <cylinder length="0.4" radius="0.05"/>
-      </geometry>
-      <origin xyz="0 0 0.2"/>
-    </collision>
-    <inertial>
-      <mass value="1.0"/>
-      <origin xyz="0 0 0.2"/>
-      <inertia ixx="0.01396" iyy="0.01396" izz="0.00125"
-        ixy="0" ixz="0" iyz="0"/>
-    </inertial>
-  </link>
-  <joint name="upper_arm_to_lower_arm" type="continuous">
-    <axis xyz="0 1 0"/>
-    <parent link="upper_arm"/>
-    <child link="lower_arm"/>
-    <origin rpy="0 0 0" xyz="0 0.1 0.35"/>
-  </joint>
-  <link name="lower_arm">
-    <visual>
-      <geometry>
-        <cylinder length="0.4" radius="0.05"/>
-      </geometry>
-      <material name="silver"/>
-      <origin xyz="0 0 0.2"/>
-    </visual>
-    <collision>
-      <geometry>
-        <cylinder length="0.4" radius="0.05"/>
-      </geometry>
-      <origin xyz="0 0 0.2"/>
-    </collision>
-    <inertial>
-      <mass value="1.0"/>
-      <origin xyz="0 0 0.2"/>
-      <inertia ixx="0.01396" iyy="0.01396" izz="0.00125"
-        ixy="0" ixz="0" iyz="0"/>
-    </inertial>
-  </link>
-  <joint name="lower_arm_to_hand" type="continuous">
-    <axis xyz="0 1 0"/>
-    <parent link="lower_arm"/>
-    <child link="hand"/>
-    <origin rpy="0 0 0" xyz="0 0 0.425"/>
-  </joint>
-  <link name="hand">
-    <visual>
-      <geometry>
-        <box size="0.05 0.05 0.05"/>
-      </geometry>
-      <material name="silver"/>
-    </visual>
-    <collision>
-      <geometry>
-        <box size="0.05 0.05 0.05"/>
-      </geometry>
-    </collision>
-    <inertial>
-      <mass value="1.0"/>
-      <inertia ixx="0.00042" iyy="0.00042" izz="0.00042"
-        ixy="0" ixz="0" iyz="0"/>
-    </inertial>
-  </link>
+    <joint name="base_joint" type="fixed">
+      <xacro:insert_block name="origin" />
+      <parent link="${parent}"/>
+      <child link="base_link"/>
+    </joint>
+    <link name="base_link">
+      <visual>
+        <geometry>
+          <cylinder length="0.05" radius="0.1"/>
+        </geometry>
+        <material name="silver"/>
+        <origin xyz="0 0 0.025"/>
+      </visual>
+      <collision>
+        <geometry>
+          <cylinder length="0.05" radius="0.1"/>
+        </geometry>
+        <origin xyz="0 0 0.025"/>
+      </collision>
+      <inertial>
+        <mass value="1.0"/>
+        <origin xyz="0 0 0.025"/>
+        <inertia ixx="0.0027" iyy="0.0027" izz="0.005" ixy="0" ixz="0" iyz="0"/>
+      </inertial>
+    </link>
+    <joint name="base_link_to_torso" type="continuous">
+      <axis xyz="0 0 1"/>
+      <parent link="base_link"/>
+      <child link="torso"/>
+      <origin rpy="0 0 0" xyz="0 0 0.05"/>
+    </joint>
+    <link name="torso">
+      <visual>
+        <geometry>
+          <cylinder length="0.5" radius="0.05"/>
+        </geometry>
+        <material name="silver"/>
+        <origin xyz="0 0 0.25"/>
+      </visual>
+      <collision>
+        <geometry>
+          <cylinder length="0.5" radius="0.05"/>
+        </geometry>
+        <origin xyz="0 0 0.25"/>
+      </collision>
+      <inertial>
+        <mass value="1.0"/>
+        <origin xyz="0 0 0.25"/>
+        <inertia ixx="0.002146" iyy="0.002146" izz="0.00125" ixy="0" ixz="0" iyz="0"/>
+      </inertial>
+    </link>
+    <joint name="torso_to_upper_arm" type="continuous">
+      <axis xyz="0 1 0"/>
+      <parent link="torso"/>
+      <child link="upper_arm"/>
+      <origin rpy="0 1.5708 0" xyz="0 -0.1 0.45"/>
+    </joint>
+    <link name="upper_arm">
+      <visual>
+        <geometry>
+          <cylinder length="0.4" radius="0.05"/>
+        </geometry>
+        <material name="silver"/>
+        <origin xyz="0 0 0.2"/>
+      </visual>
+      <collision>
+        <geometry>
+          <cylinder length="0.4" radius="0.05"/>
+        </geometry>
+        <origin xyz="0 0 0.2"/>
+      </collision>
+      <inertial>
+        <mass value="1.0"/>
+        <origin xyz="0 0 0.2"/>
+        <inertia ixx="0.01396" iyy="0.01396" izz="0.00125" ixy="0" ixz="0" iyz="0"/>
+      </inertial>
+    </link>
+    <joint name="upper_arm_to_lower_arm" type="continuous">
+      <axis xyz="0 1 0"/>
+      <parent link="upper_arm"/>
+      <child link="lower_arm"/>
+      <origin rpy="0 0 0" xyz="0 0.1 0.35"/>
+    </joint>
+    <link name="lower_arm">
+      <visual>
+        <geometry>
+          <cylinder length="0.4" radius="0.05"/>
+        </geometry>
+        <material name="silver"/>
+        <origin xyz="0 0 0.2"/>
+      </visual>
+      <collision>
+        <geometry>
+          <cylinder length="0.4" radius="0.05"/>
+        </geometry>
+        <origin xyz="0 0 0.2"/>
+      </collision>
+      <inertial>
+        <mass value="1.0"/>
+        <origin xyz="0 0 0.2"/>
+        <inertia ixx="0.01396" iyy="0.01396" izz="0.00125" ixy="0" ixz="0" iyz="0"/>
+      </inertial>
+    </link>
+    <joint name="lower_arm_to_hand" type="continuous">
+      <axis xyz="0 1 0"/>
+      <parent link="lower_arm"/>
+      <child link="hand"/>
+      <origin rpy="0 0 0" xyz="0 0 0.425"/>
+    </joint>
+    <link name="hand">
+      <visual>
+        <geometry>
+          <box size="0.05 0.05 0.05"/>
+        </geometry>
+        <material name="silver"/>
+      </visual>
+      <collision>
+        <geometry>
+          <box size="0.05 0.05 0.05"/>
+        </geometry>
+      </collision>
+      <inertial>
+        <mass value="1.0"/>
+        <inertia ixx="0.00042" iyy="0.00042" izz="0.00042" ixy="0" ixz="0" iyz="0"/>
+      </inertial>
+    </link>
   </xacro:macro>
 </robot>
