Commit message: New model for pinchy from onshape CAD drawing

File: pinchy_robot/pinchy_robot_description/models/pinchy.ros2_control copy.xacro (robot description, xacro)
@@ -14,5 +14,5 @@
                 </xacro:unless>
             </hardware>
-            <joint name="013_011_continuous">
+            <joint name="base_link_to_torso">
                 <command_interface name="position">
                     <param name="min">-1</param>
@@ -21,5 +21,5 @@
                 <state_interface name="position"/>
             </joint>
-            <joint name="base_varm">
+            <joint name="torso_to_upper_arm">
                 <command_interface name="position">
                     <param name="min">-1</param>
@@ -28,5 +28,12 @@
                 <state_interface name="position"/>
             </joint>
-            <joint name="base_mainarm">
+            <joint name="upper_arm_to_lower_arm">
+                <command_interface name="position">
+                    <param name="min">-1</param>
+                    <param name="max">1</param>
+                </command_interface>
+                <state_interface name="position"/>
+            </joint>
+            <joint name="lower_arm_to_hand">
                 <command_interface name="position">
                     <param name="min">-1</param>
