Commit message: New model for pinchy from onshape CAD drawing

File: pinchy_robot/pinchy_robot_description/models/pinchy_onshape.urdf.xacro (robot description, xacro)
@@ -24,7 +24,7 @@
             </collision>
             <inertial>
-                <origin xyz="-0.033485894275804402309 -1.2001011211791619353e-09 0.021753373316492456702" rpy="0 0 0"/>
+                <origin xyz="-0.033485894275804409248 -1.2001011143591475339e-09 0.021753373316492453232" rpy="0 0 0"/>
                 <mass value="0.11759175314133056556" />
-                <inertia ixx="0.00010757491305669516222" ixy="9.6951976383166017242e-12" ixz="-1.129955118934984161e-05" iyy="0.00028157118801149162062" iyz="-1.1113073360885274726e-12" izz="0.00033120803272819855992" />
+                <inertia ixx="0.00010757491305669513511" ixy="9.6951976338254601312e-12" ixz="-1.1299551189349826363e-05" iyy="0.00028157118801149167483" iyz="-1.1113073401130564013e-12" izz="0.00033120803272819866834" />
             </inertial>
         </link>
@@ -48,10 +48,10 @@
                 <origin xyz="0.038334151784957443132 0.023999999999999774986 -0.003861060291331577278" rpy="0 0 0"/>
                 <mass value="0.050632060796438636829" />
-                <inertia ixx="2.3412926852668567671e-05" ixy="0" ixz="-5.1918600718263601986e-09" iyy="2.418011164816487058e-05" iyz="0" izz="4.7075071061242765649e-05" />
+                <inertia ixx="2.3412926852668577835e-05" ixy="0" ixz="-5.1918600718263734335e-09" iyy="2.418011164816487058e-05" iyz="0" izz="4.7075071061242765649e-05" />
             </inertial>
         </link>
         <link name="011_gearmast">
             <visual>
-                <origin xyz="-3.0814879110195773649e-33 0 0.00074118095489748153648" rpy="-1.570796326794896558 -1.9721522630525290756e-31 2.8808654239159165536e-18" />
+                <origin xyz="0 1.5407439555097886824e-33 0.00074118095489748153648" rpy="-1.570796326794896558 -3.0814879110195773649e-33 -8.1652472595093291124e-20" />
                 <geometry>
                     <mesh filename="package://pinchy_robot_description/models/mesh/011_gearmast.stl"/>
@@ -62,5 +62,5 @@
             </visual>
             <collision>
-                <origin xyz="-3.0814879110195773649e-33 0 0.00074118095489748153648" rpy="-1.570796326794896558 -1.9721522630525290756e-31 2.8808654239159165536e-18" />
+                <origin xyz="0 1.5407439555097886824e-33 0.00074118095489748153648" rpy="-1.570796326794896558 -3.0814879110195773649e-33 -8.1652472595093291124e-20" />
                 <geometry>
                     <mesh filename="package://pinchy_robot_description/models/mesh/011_gearmast.stl"/>
@@ -68,12 +68,12 @@
             </collision>
             <inertial>
-                <origin xyz="0.0011448146623121613526 -4.5614544122798960911e-08 0.0043556640618009276333" rpy="0 0 0"/>
+                <origin xyz="0.0011448146623121611357 -4.5614544123273696408e-08 0.0043556640618009276333" rpy="0 0 0"/>
                 <mass value="0.037429445757737357658" />
-                <inertia ixx="1.3678283742239876844e-05" ixy="-1.8558228083068321185e-12" ixz="4.9208020155399961048e-09" iyy="1.3452672074635373909e-05" iyz="-8.9136290706351023319e-13" izz="2.6827475442753630485e-05" />
+                <inertia ixx="1.3678283742239870068e-05" ixy="-1.8558228082889677638e-12" ixz="4.920802015539978734e-09" iyy="1.3452672074635370521e-05" iyz="-8.9136290706678028252e-13" izz="2.6827475442753623709e-05" />
             </inertial>
         </link>
         <link name="001_base">
             <visual>
-                <origin xyz="-5.5059794306154815924e-18 -2.5229826121639363311e-20 0" rpy="3.141592653589793116 -0 1.292162160811374467e-17" />
+                <origin xyz="-5.505979430618637036e-18 -2.5229826121047717632e-20 0" rpy="3.141592653589793116 -0 -1.1363109399182029424e-17" />
                 <geometry>
                     <mesh filename="package://pinchy_robot_description/models/mesh/001_base.stl"/>
@@ -84,5 +84,5 @@
             </visual>
             <collision>
-                <origin xyz="-5.5059794306154815924e-18 -2.5229826121639363311e-20 0" rpy="3.141592653589793116 -0 1.292162160811374467e-17" />
+                <origin xyz="-5.505979430618637036e-18 -2.5229826121047717632e-20 0" rpy="3.141592653589793116 -0 -1.1363109399182029424e-17" />
                 <geometry>
                     <mesh filename="package://pinchy_robot_description/models/mesh/001_base.stl"/>
@@ -90,59 +90,269 @@
             </collision>
             <inertial>
-                <origin xyz="0.001161673545557385728 0.00092317800064807868047 -0.020499360341960613796" rpy="0 0 0"/>
-                <mass value="0.17975423326260306367" />
-                <inertia ixx="0.00012231885879902305598" ixy="-3.4507707064030143545e-06" ixz="5.818271012981028621e-06" iyy="0.00012893735685722983089" iyz="5.8342500739731076949e-06" izz="0.00014275976070929840243" />
-            </inertial>
-        </link>
-        <link name="closing_001_005_2">
+                <origin xyz="0.001161673545557385728 0.00092317800064807998151 -0.020499360341960603388" rpy="0 0 0"/>
+                <mass value="0.17975423326260300816" />
+                <inertia ixx="0.00012231885879902300177" ixy="-3.4507707064030173191e-06" ixz="5.8182710129810311621e-06" iyy="0.00012893735685722983089" iyz="5.8342500739731093889e-06" izz="0.00014275976070929840243" />
+            </inertial>
+        </link>
+        <link name="003_varm">
+            <visual>
+                <origin xyz="3.4694469519536141888e-18 0 0" rpy="2.9422690944093511222e-18 -1.2079259381544499194e-17 -3.3026307202013133133e-17" />
+                <geometry>
+                    <mesh filename="package://pinchy_robot_description/models/mesh/003_varm.stl"/>
+                </geometry>
+                <material name="003_varm_material">
+                    <color rgba="0.84313725490196078649 0.35294117647058825815 0 1.0"/>
+                </material>
+            </visual>
+            <collision>
+                <origin xyz="3.4694469519536141888e-18 0 0" rpy="2.9422690944093511222e-18 -1.2079259381544499194e-17 -3.3026307202013133133e-17" />
+                <geometry>
+                    <mesh filename="package://pinchy_robot_description/models/mesh/003_varm.stl"/>
+                </geometry>
+            </collision>
+            <inertial>
+                <origin xyz="0.020430554246132631713 0.00055877620043398080509 0.0054371933906984196844" rpy="0 0 0"/>
+                <mass value="0.015276016785753359847" />
+                <inertia ixx="7.9306883740486619467e-07" ixy="-1.3538496626389062662e-07" ixz="-4.2655352640383100139e-07" iyy="6.6187561149688310921e-06" iyz="-9.1660691416123494077e-09" izz="6.935882283253827984e-06" />
+            </inertial>
+        </link>
+        <link name="004_link_135">
+            <visual>
+                <origin xyz="-0.067499999999999976685 3.4694469519536141888e-18 -0.005500000000000004885" rpy="-8.3612752561080595641e-18 1.1204020728012776145e-18 -4.6293373202296152882e-17" />
+                <geometry>
+                    <mesh filename="package://pinchy_robot_description/models/mesh/004_link_135.stl"/>
+                </geometry>
+                <material name="004_link_135_material">
+                    <color rgba="0.84313725490196078649 0.35294117647058825815 0 1.0"/>
+                </material>
+            </visual>
+            <collision>
+                <origin xyz="-0.067499999999999976685 3.4694469519536141888e-18 -0.005500000000000004885" rpy="-8.3612752561080595641e-18 1.1204020728012776145e-18 -4.6293373202296152882e-17" />
+                <geometry>
+                    <mesh filename="package://pinchy_robot_description/models/mesh/004_link_135.stl"/>
+                </geometry>
+            </collision>
+            <inertial>
+                <origin xyz="-0.073433819965337529534 7.4331604101003543475e-06 -0.0028218133227464218746" rpy="0 0 0"/>
+                <mass value="0.007392576800685658929" />
+                <inertia ixx="8.4434163215744383027e-08" ixy="-3.185208938332878106e-10" ixz="2.1645499427877073862e-07" iyy="1.6665438826907819157e-05" iyz="1.3976046566816867928e-10" izz="1.6683971677717033204e-05" />
+            </inertial>
+        </link>
+        <link name="006_horarm">
+            <visual>
+                <origin xyz="0.056999999999999939604 0 -0.0099500000000000039801" rpy="1.570796326794896558 2.3420334037882265916e-17 2.5063458259735427873e-18" />
+                <geometry>
+                    <mesh filename="package://pinchy_robot_description/models/mesh/006_horarm.stl"/>
+                </geometry>
+                <material name="006_horarm_material">
+                    <color rgba="0.84313725490196078649 0.35294117647058825815 0 1.0"/>
+                </material>
+            </visual>
+            <collision>
+                <origin xyz="0.056999999999999939604 0 -0.0099500000000000039801" rpy="1.570796326794896558 2.3420334037882265916e-17 2.5063458259735427873e-18" />
+                <geometry>
+                    <mesh filename="package://pinchy_robot_description/models/mesh/006_horarm.stl"/>
+                </geometry>
+            </collision>
+            <inertial>
+                <origin xyz="0.094081019082547429067 -0.012440624561642035784 -0.011734173613708449163" rpy="0 0 0"/>
+                <mass value="0.048591753045881112827" />
+                <inertia ixx="6.9180719655106513242e-06" ixy="-7.7587950973339834449e-07" ixz="5.5264376053445264962e-06" iyy="0.0001734130847172764083" iyz="-5.8856462243627846272e-07" izz="0.00017375882723609468723" />
+            </inertial>
+        </link>
+        <link name="closing_002_006_1">
             <inertial>
                 <origin xyz="0 0 0" rpy="0 0 0" />
                 <mass value="1e-9" />
-                <inertia ixx="0" ixy="0" ixz="0" iyy="0" iyz="0" izz="0" />
-            </inertial>
-        </link>
-        <joint name="closing_001_005_2_frame" type="fixed">
-            <origin xyz="0.027999999999999986705 0.037969999999999996809 -0.063189999999999996172" rpy="1.2921621608113746211e-17 -1.570796326794896558 0" />
-            <parent link="001_base" />
-            <child link="closing_001_005_2" />
-            <axis xyz="0 0 0"/>
-        </joint>
-        <link name="003_varm">
-            <visual>
-                <origin xyz="0 1.3877787807814456755e-17 0" rpy="-5.4702925957144849332e-18 1.9477237810650893854e-18 -2.7565511512361946476e-17" />
-                <geometry>
-                    <mesh filename="package://pinchy_robot_description/models/mesh/003_varm.stl"/>
-                </geometry>
-                <material name="003_varm_material">
-                    <color rgba="0.84313725490196078649 0.35294117647058825815 0 1.0"/>
-                </material>
-            </visual>
-            <collision>
-                <origin xyz="0 1.3877787807814456755e-17 0" rpy="-5.4702925957144849332e-18 1.9477237810650893854e-18 -2.7565511512361946476e-17" />
-                <geometry>
-                    <mesh filename="package://pinchy_robot_description/models/mesh/003_varm.stl"/>
-                </geometry>
-            </collision>
-            <inertial>
-                <origin xyz="0.020430554246132628243 0.00055877620043399446603 0.0054371933906984196844" rpy="0 0 0"/>
-                <mass value="0.015276016785753359847" />
-                <inertia ixx="7.9306883740486598291e-07" ixy="-1.3538496626389067956e-07" ixz="-4.2655352640383078964e-07" iyy="6.6187561149688319391e-06" iyz="-9.1660691416123990385e-09" izz="6.935882283253829678e-06" />
-            </inertial>
-        </link>
-        <link name="closing_003_004_2">
+                <inertia ixx="2.4030086788760112591e-06" ixy="-1.3882584188564426332e-07" ixz="-3.4438410484124220848e-08" iyy="8.1820709705349406091e-06" iyz="-2.9879442802538686064e-07" izz="9.3619592049011330812e-06" />
+            </inertial>
+        </link>
+        <joint name="closing_002_006_1_frame" type="fixed">
+            <origin xyz="0.056999999999999925726 0 -0.016950000000000013667" rpy="1.6668858177201397623e-18 2.3420334037882265916e-17 2.5063458259735427873e-18" />
+            <parent link="006_horarm" />
+            <child link="closing_002_006_1" />
+            <axis xyz="0 0 1"/>
+        </joint>
+        <link name="009_trialinkfront">
+            <visual>
+                <origin xyz="-0.039299999999999987721 -0.0065000000000000335287 0" rpy="-1.570796326794896558 -1.570796326794896558 0" />
+                <geometry>
+                    <mesh filename="package://pinchy_robot_description/models/mesh/009_trialinkfront.stl"/>
+                </geometry>
+                <material name="009_trialinkfront_material">
+                    <color rgba="0.84313725490196078649 0.35294117647058825815 0 1.0"/>
+                </material>
+            </visual>
+            <collision>
+                <origin xyz="-0.039299999999999987721 -0.0065000000000000335287 0" rpy="-1.570796326794896558 -1.570796326794896558 0" />
+                <geometry>
+                    <mesh filename="package://pinchy_robot_description/models/mesh/009_trialinkfront.stl"/>
+                </geometry>
+            </collision>
+            <inertial>
+                <origin xyz="-0.023138260045836366724 0.0096562717419969509858 -0.0090452320899661597942" rpy="0 0 0"/>
+                <mass value="0.018960886227135643339" />
+                <inertia ixx="3.3194985728346417554e-06" ixy="1.12998941383453901e-06" ixz="-3.2618401827615369512e-07" iyy="3.1952109322463258382e-06" iyz="3.7054522324610349251e-07" izz="5.2884049184070589409e-06" />
+            </inertial>
+        </link>
+        <link name="closing_008_009_1">
             <inertial>
                 <origin xyz="0 0 0" rpy="0 0 0" />
                 <mass value="1e-9" />
-                <inertia ixx="0" ixy="0" ixz="0" iyy="0" iyz="0" izz="0" />
-            </inertial>
-        </link>
-        <joint name="closing_003_004_2_frame" type="fixed">
-            <origin xyz="0.056999999999999995115 1.3877787807814456755e-17 0.0050000000000000044409" rpy="1.7743817425140666063e-16 -5.4702925957144849332e-18 -1.570796326794896558" />
+                <inertia ixx="2.4030086788760112591e-06" ixy="-1.3882584188564426332e-07" ixz="-3.4438410484124220848e-08" iyy="8.1820709705349406091e-06" iyz="-2.9879442802538686064e-07" izz="9.3619592049011330812e-06" />
+            </inertial>
+        </link>
+        <joint name="closing_008_009_1_frame" type="fixed">
+            <origin xyz="-0.032799999999999981948 0.028499999999999969802 -0.021999999999999991784" rpy="3.141592653589793116 2.8263439549994856564e-17 -3.773070744741489802e-20" />
+            <parent link="009_trialinkfront" />
+            <child link="closing_008_009_1" />
+            <axis xyz="0 0 1"/>
+        </joint>
+        <link name="014_clawbase">
+            <visual>
+                <origin xyz="-0.0017000000000000009895 0.020300000000000012479 -0.0060000000000000053291" rpy="1.570796326794896558 1.570796326794896558 0" />
+                <geometry>
+                    <mesh filename="package://pinchy_robot_description/models/mesh/014_clawbase.stl"/>
+                </geometry>
+                <material name="014_clawbase_material">
+                    <color rgba="0.84313725490196078649 0.35294117647058825815 0 1.0"/>
+                </material>
+            </visual>
+            <collision>
+                <origin xyz="-0.0017000000000000009895 0.020300000000000012479 -0.0060000000000000053291" rpy="1.570796326794896558 1.570796326794896558 0" />
+                <geometry>
+                    <mesh filename="package://pinchy_robot_description/models/mesh/014_clawbase.stl"/>
+                </geometry>
+            </collision>
+            <inertial>
+                <origin xyz="-0.0018790345340905676916 0.012684764644607016484 -0.012449562627841494894" rpy="0 0 0"/>
+                <mass value="0.01015928222090070436" />
+                <inertia ixx="2.8161631051851268062e-06" ixy="-2.0681515990841533094e-08" ixz="2.6448338684182113098e-08" iyy="2.8740865083613729631e-06" iyz="5.3943746192763651611e-07" izz="1.0774908755333261357e-06" />
+            </inertial>
+        </link>
+        <link name="015_clawfingerdx">
+            <visual>
+                <origin xyz="0 1.7347234759768070944e-18 -0.00029999999999999471534" rpy="1.570796326794896558 -3.8283574422962246717e-19 -2.5828392060750557018e-18" />
+                <geometry>
+                    <mesh filename="package://pinchy_robot_description/models/mesh/015_clawfingerdx.stl"/>
+                </geometry>
+                <material name="015_clawfingerdx_material">
+                    <color rgba="0.84313725490196078649 0.35294117647058825815 0 1.0"/>
+                </material>
+            </visual>
+            <collision>
+                <origin xyz="0 1.7347234759768070944e-18 -0.00029999999999999471534" rpy="1.570796326794896558 -3.8283574422962246717e-19 -2.5828392060750557018e-18" />
+                <geometry>
+                    <mesh filename="package://pinchy_robot_description/models/mesh/015_clawfingerdx.stl"/>
+                </geometry>
+            </collision>
+            <inertial>
+                <origin xyz="0.018455747659032673696 0.0025339063026478796797 -0.0012325548331221657279" rpy="0 0 0"/>
+                <mass value="0.0017886183280535160583" />
+                <inertia ixx="2.7268812321605331177e-08" ixy="-3.5813623681470532009e-08" ixz="-1.9991865655434482958e-08" iyy="5.1662283716070205294e-07" iyz="-4.5698409967013661735e-09" izz="5.3293341889482562252e-07" />
+            </inertial>
+        </link>
+        <joint name="014_015" type="fixed">
+            <origin xyz="-0.01074999999999999567 0.020300000000000040234 -0.01450000000000031819" rpy="1.57079632679489678 1.5707963267948954478 0" />
+            <parent link="014_clawbase" />
+            <child link="015_clawfingerdx" />
+            <axis xyz="0 0 1"/>
+            <limit effort="1" velocity="20" />
+            <joint_properties friction="0.0"/>
+        </joint>
+        <link name="017_clawfingersx">
+            <visual>
+                <origin xyz="0 -1.7347234759768070944e-18 -0.0032999999999999973799" rpy="-1.570796326794896558 1.91290401938423627e-19 -1.0336689845248326166e-19" />
+                <geometry>
+                    <mesh filename="package://pinchy_robot_description/models/mesh/017_clawfingersx.stl"/>
+                </geometry>
+                <material name="017_clawfingersx_material">
+                    <color rgba="0.84313725490196078649 0.35294117647058825815 0 1.0"/>
+                </material>
+            </visual>
+            <collision>
+                <origin xyz="0 -1.7347234759768070944e-18 -0.0032999999999999973799" rpy="-1.570796326794896558 1.91290401938423627e-19 -1.0336689845248326166e-19" />
+                <geometry>
+                    <mesh filename="package://pinchy_robot_description/models/mesh/017_clawfingersx.stl"/>
+                </geometry>
+            </collision>
+            <inertial>
+                <origin xyz="0.01881208674862810612 -0.0025600078614870800178 -0.0012092355891364032008" rpy="0 0 0"/>
+                <mass value="0.0017289482656387797528" />
+                <inertia ixx="2.6945353811716051557e-08" ixy="3.4907708389775138057e-08" ixz="-1.8961027589390282731e-08" iyy="5.0190649161374519976e-07" iyz="4.4234371214567529165e-09" izz="5.1825789788917879662e-07" />
+            </inertial>
+        </link>
+        <link name="018_clawgeardriven">
+            <visual>
+                <origin xyz="-2.7755575615628913511e-17 -1.7347234759768070944e-18 -0.0049999999999999766853" rpy="-1.570796326794896558 -1.9101089742314066949e-19 1.6125877135095972468e-17" />
+                <geometry>
+                    <mesh filename="package://pinchy_robot_description/models/mesh/018_clawgeardriven.stl"/>
+                </geometry>
+                <material name="018_clawgeardriven_material">
+                    <color rgba="0.84313725490196078649 0.35294117647058825815 0 1.0"/>
+                </material>
+            </visual>
+            <collision>
+                <origin xyz="-2.7755575615628913511e-17 -1.7347234759768070944e-18 -0.0049999999999999766853" rpy="-1.570796326794896558 -1.9101089742314066949e-19 1.6125877135095972468e-17" />
+                <geometry>
+                    <mesh filename="package://pinchy_robot_description/models/mesh/018_clawgeardriven.stl"/>
+                </geometry>
+            </collision>
+            <inertial>
+                <origin xyz="-1.7230839811980370275e-06 0.0016346299156224134656 -0.0025169330447530301187" rpy="0 0 0"/>
+                <mass value="0.0016432484276812276032" />
+                <inertia ixx="4.3940469046301066529e-08" ixy="9.2068379919175633376e-12" ixz="-1.6487089256642451513e-12" iyy="4.3401024087893505717e-08" iyz="4.7246181535537862836e-09" izz="7.8152690487289344876e-08" />
+            </inertial>
+        </link>
+        <joint name="017_018" type="fixed">
+            <origin xyz="-2.7755575615628913511e-17 -8.3266726846886740532e-17 -0.0032999999999999696243" rpy="-3.0263178583034298145e-16 -4.4860140403825905728e-17 -3.1415926535897917837" />
+            <parent link="017_clawfingersx" />
+            <child link="018_clawgeardriven" />
+            <axis xyz="0 0 1"/>
+            <limit effort="1" velocity="20" />
+            <joint_properties friction="0.0"/>
+        </joint>
+        <joint name="014_017" type="fixed">
+            <origin xyz="0.0073500000000000648148 0.020300000000000012479 -0.014500000000000040634" rpy="1.570796326794896558 1.570796326794896336 0" />
+            <parent link="014_clawbase" />
+            <child link="017_clawfingersx" />
+            <axis xyz="0 0 1"/>
+            <limit effort="1" velocity="20" />
+            <joint_properties friction="0.0"/>
+        </joint>
+        <joint name="009_014" type="fixed">
+            <origin xyz="-0.039299999999999835065 0.010849999999999915268 -0.0069999999999999836658" rpy="3.141592653589793116 -1.570796326794896558 0" />
+            <parent link="009_trialinkfront" />
+            <child link="014_clawbase" />
+            <axis xyz="0 0 1"/>
+            <limit effort="1" velocity="20" />
+            <joint_properties friction="0.0"/>
+        </joint>
+        <joint name="006_009" type="revolute">
+            <origin xyz="0.20399999999999943179 1.1102230246251565404e-16 -0.0079499999999998773037" rpy="-4.2119620857286530011e-15 5.3426477407382402562e-15 2.9724702659122148596" />
+            <parent link="006_horarm" />
+            <child link="009_trialinkfront" />
+            <axis xyz="0 0 1"/>
+            <limit effort="1" velocity="20" lower="-3.141592653589793116" upper="3.141592653589793116"/>
+            <joint_properties friction="0.0"/>
+        </joint>
+        <joint name="link_135_horarm" type="revolute">
+            <origin xyz="-0.1350000000000001199 5.273559366969493567e-16 -0.0054999999999999008016" rpy="2.0578910659424728341e-15 4.3162916163402126325e-15 -0.92649077294944326422" />
+            <parent link="004_link_135" />
+            <child link="006_horarm" />
+            <axis xyz="0 0 1"/>
+            <limit effort="1" velocity="20" lower="-3.141592653589793116" upper="3.141592653589793116"/>
+            <joint_properties friction="0.0"/>
+        </joint>
+        <joint name="varm_link_135" type="revolute">
+            <origin xyz="0.056999999999999960421 -2.7755575615628913511e-17 0.010450000000001149342" rpy="-1.0166412649775068718e-14 -3.0576035131021497408e-15 -2.2151018806402720251" />
             <parent link="003_varm" />
-            <child link="closing_003_004_2" />
-            <axis xyz="0 0 0"/>
-        </joint>
-        <joint name="001_003" type="revolute">
-            <origin xyz="-0.012499999999999976408 3.1170380091756358422e-17 -0.043000000000000072886" rpy="-1.5707963267948961139 -0.34187976534138431184 1.570796326794891451" />
+            <child link="004_link_135" />
+            <axis xyz="0 0 1"/>
+            <limit effort="1" velocity="20" lower="-3.141592653589793116" upper="3.141592653589793116"/>
+            <joint_properties friction="0.0"/>
+        </joint>
+        <joint name="base_varm" type="revolute">
+            <origin xyz="-0.012499999999999986816 7.1053158380719087885e-18 -0.042999999999999968803" rpy="-1.570796326794896336 0.16553213915207776186 1.5707963267949005548" />
             <parent link="001_base" />
             <child link="003_varm" />
@@ -153,5 +363,5 @@
         <link name="002_mainarm">
             <visual>
-                <origin xyz="-1.084202172485504434e-19 0 0.0082500000000000003886" rpy="-1.570796326794896558 2.1823454752613109057e-18 3.3366817323438506917e-19" />
+                <origin xyz="0 0 0.0082500000000000003886" rpy="-1.570796326794896558 1.8855661413192599729e-17 -6.6499555712529986536e-19" />
                 <geometry>
                     <mesh filename="package://pinchy_robot_description/models/mesh/002_mainarm.stl"/>
@@ -162,5 +372,5 @@
             </visual>
             <collision>
-                <origin xyz="-1.084202172485504434e-19 0 0.0082500000000000003886" rpy="-1.570796326794896558 2.1823454752613109057e-18 3.3366817323438506917e-19" />
+                <origin xyz="0 0 0.0082500000000000003886" rpy="-1.570796326794896558 1.8855661413192599729e-17 -6.6499555712529986536e-19" />
                 <geometry>
                     <mesh filename="package://pinchy_robot_description/models/mesh/002_mainarm.stl"/>
@@ -168,371 +378,161 @@
             </collision>
             <inertial>
-                <origin xyz="-0.0045289479351360746595 0.058063314437010481173 0.010438692473920995613" rpy="0 0 0"/>
-                <mass value="0.089768612982453629967" />
-                <inertia ixx="0.0001937977516965140091" ixy="1.4539001404579357045e-06" ixz="4.0937771123815081593e-07" iyy="1.5304948332152038372e-05" iyz="-1.0315307235679156346e-06" izz="0.00019169602556341142964" />
-            </inertial>
-        </link>
-        <link name="006_horarm">
-            <visual>
-                <origin xyz="-1.3877787807814456755e-17 5.5511151231257827021e-17 0.0070000000000000096867" rpy="1.570796326794896558 -4.5456754938217338643e-18 2.7501720434233651453e-17" />
-                <geometry>
-                    <mesh filename="package://pinchy_robot_description/models/mesh/006_horarm.stl"/>
-                </geometry>
-                <material name="006_horarm_material">
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